File: Project/IO Expander.kicad_sch (KiCad schematic)
At the start: 32 parts, among them J801 Conn_02x08_Odd_Even, U801 MCP23017T-E_ML

Commit message: More files cleanup
Other:
- company: Quasi Peak -> ${COMPANY}
