File: Project/Microcontroller.kicad_sch (KiCad schematic)
At the start: 22 parts, among them J701 Conn_01x05_Female, J702 Conn_01x04_Female, J703 Conn_01x04_Female, U701 STM32L031K6U3TR

Commit message: More files cleanup
Other:
- company: Quasi Peak -> ${COMPANY}
Changed lines of the file:
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@@
     (title "TMC6200-TA-T Eval Board")
     (date "2021-09-03")
-    (rev "ED A0")
-    (company "Quasi Peak")
-    (comment 1 "Patryk Rzońca")
+    (rev "${REVISION}")
+    (company "${COMPANY}")
+    (comment 1 "${ENGINEER}")
+    (comment 2 "${PHONE_NUMBER}")
+    (comment 3 "${EMAIL}")
+    (comment 4 "${SENTENCE}")
   )
   (junction (at 147.32 133.35) (diameter 0) (color 0 0 0 0)
@@
     (pin "9")
   )
-  (symbol (lib_id "Device:C") (at 36.83 52.07 0) (mirror x)
+  (symbol (lib_id "Device:C") (at 36.83 52.07 0) (mirror x) (unit 1)
     (in_bom yes) (on_board yes)
     (property "Reference" "C701" (id 0) (at 31.115 50.8 0)
@@
     (pin "2")
   )
-  (symbol (lib_id "Device:C") (at 34.925 74.295 0) (mirror x)
+  (symbol (lib_id "Device:C") (at 34.925 74.295 0) (mirror x) (unit 1)
     (in_bom yes) (on_board yes)
     (property "Reference" "C704" (id 0) (at 29.21 73.025 0)
@@
     (pin "2")
   )
-  (symbol (lib_id "Device:C") (at 45.72 52.07 0)
+  (symbol (lib_id "Device:C") (at 45.72 52.07 0) (unit 1)
     (in_bom yes) (on_board yes)
     (property "Reference" "C702" (id 0) (at 40.005 50.8 0)
@@
     (pin "2")
   )
-  (symbol (lib_id "Device:C") (at 54.61 52.07 0)
+  (symbol (lib_id "Device:C") (at 54.61 52.07 0) (unit 1)
     (in_bom yes) (on_board yes)
     (property "Reference" "C703" (id 0) (at 48.895 50.8 0)
@@
     (pin "2")
   )
-  (symbol (lib_id "Device:C") (at 49.53 74.295 0)
+  (symbol (lib_id "Device:C") (at 49.53 74.295 0) (unit 1)
     (in_bom yes) (on_board yes)
     (property "Reference" "C705" (id 0) (at 43.815 73.025 0)
@@
     (pin "2")
   )
-  (symbol (lib_id "power:+3.3V") (at 26.67 44.45 0)
+  (symbol (lib_id "power:+3.3V") (at 26.67 44.45 0) (unit 1)
     (in_bom yes) (on_board yes)
     (property "Reference" "#PWR0704" (id 0) (at 26.67 48.26 0)
@@
     (pin "1")
   )
-  (symbol (lib_id "power:+3.3V") (at 31.115 67.945 0)
+  (symbol (lib_id "power:+3.3V") (at 31.115 67.945 0) (unit 1)
     (in_bom yes) (on_board yes)
     (property "Reference" "#PWR0711" (id 0) (at 31.115 71.755 0)
@@
     (pin "1")
   )
-  (symbol (lib_id "power:GND") (at 197.485 79.375 0) (mirror y)
+  (symbol (lib_id "power:GND") (at 197.485 79.375 0) (mirror y) (unit 1)
     (in_bom yes) (on_board yes)
     (property "Reference" "#PWR0715" (id 0) (at 197.485 85.725 0)
@@
     (pin "1")
   )
-  (symbol (lib_id "power:GND") (at 36.83 57.15 0) (mirror y)
+  (symbol (lib_id "power:GND") (at 36.83 57.15 0) (mirror y) (unit 1)
     (in_bom yes) (on_board yes)
     (property "Reference" "#PWR0708" (id 0) (at 36.83 63.5 0)
@@
     (pin "1")
   )
-  (symbol (lib_id "power:GND") (at 45.72 57.15 0) (mirror y)
+  (symbol (lib_id "power:GND") (at 45.72 57.15 0) (mirror y) (unit 1)
     (in_bom yes) (on_board yes)
     (property "Reference" "#PWR0709" (id 0) (at 45.72 63.5 0)
@@
     (pin "1")
   )
-  (symbol (lib_id "power:GND") (at 54.61 57.15 0) (mirror y)
+  (symbol (lib_id "power:GND") (at 54.61 57.15 0) (mirror y) (unit 1)
     (in_bom yes) (on_board yes)
     (property "Reference" "#PWR0710" (id 0) (at 54.61 63.5 0)
@@
     (pin "1")
   )
-  (symbol (lib_id "power:GND") (at 49.53 79.375 0) (mirror y)
+  (symbol (lib_id "power:GND") (at 49.53 79.375 0) (mirror y) (unit 1)
     (in_bom yes) (on_board yes)
     (property "Reference" "#PWR0714" (id 0) (at 49.53 85.725 0)
@@
     (pin "1")
   )
-  (symbol (lib_id "power:GND") (at 34.925 79.375 0) (mirror y)
+  (symbol (lib_id "power:GND") (at 34.925 79.375 0) (mirror y) (unit 1)
     (in_bom yes) (on_board yes)
     (property "Reference" "#PWR0713" (id 0) (at 34.925 85.725 0)
@@
     (pin "1")
   )
-  (symbol (lib_id "power:GND") (at 147.32 143.51 0) (mirror y)
+  (symbol (lib_id "power:GND") (at 147.32 143.51 0) (mirror y) (unit 1)
     (in_bom yes) (on_board yes)
     (property "Reference" "#PWR0721" (id 0) (at 147.32 149.86 0)
@@
     (pin "1")
   )
-  (symbol (lib_id "Device:C") (at 147.32 138.43 0)
+  (symbol (lib_id "Device:C") (at 147.32 138.43 0) (unit 1)
     (in_bom yes) (on_board yes)
     (property "Reference" "C706" (id 0) (at 141.605 137.16 0)
@@
     (pin "2")
   )
-  (symbol (lib_id "Device:R") (at 147.32 128.27 0) (mirror x)
+  (symbol (lib_id "Device:R") (at 147.32 128.27 0) (mirror x) (unit 1)
     (in_bom yes) (on_board yes)
     (property "Reference" "R704" (id 0) (at 141.605 126.365 0)
@@
     (pin "1")
   )
-  (symbol (lib_id "power:GND") (at 142.24 55.245 0) (mirror y)
+  (symbol (lib_id "power:GND") (at 142.24 55.245 0) (mirror y) (unit 1)
     (in_bom yes) (on_board yes)
     (property "Reference" "#PWR0707" (id 0) (at 142.24 61.595 0)
@@
     (pin "1")
   )
-  (symbol (lib_id "Device:R") (at 31.75 46.99 270) (mirror x)
+  (symbol (lib_id "Device:R") (at 31.75 46.99 270) (mirror x) (unit 1)
     (in_bom yes) (on_board yes)
     (property "Reference" "R701" (id 0) (at 29.21 43.815 90)
@@
     (pin "2")
   )
-  (symbol (lib_id "Device:LED") (at 254 138.43 90)
+  (symbol (lib_id "Device:LED") (at 254 138.43 90) (unit 1)
     (in_bom yes) (on_board yes)
     (property "Reference" "D701" (id 0) (at 248.92 137.16 90)
@@
     (pin "2")
   )
-  (symbol (lib_id "Device:R") (at 254 129.54 0) (mirror x)
+  (symbol (lib_id "Device:R") (at 254 129.54 0) (mirror x) (unit 1)
     (in_bom yes) (on_board yes)
     (property "Reference" "R705" (id 0) (at 248.285 127.635 0)
@@
     (pin "1")
   )
-  (symbol (lib_id "power:GND") (at 101.6 143.51 0) (mirror y)
+  (symbol (lib_id "power:GND") (at 101.6 143.51 0) (mirror y) (unit 1)
     (in_bom yes) (on_board yes)
     (property "Reference" "#PWR0720" (id 0) (at 101.6 149.86 0)
@@
     (pin "1")
   )
-  (symbol (lib_id "power:+3.3V") (at 101.6 130.81 0)
+  (symbol (lib_id "power:+3.3V") (at 101.6 130.81 0) (unit 1)
     (in_bom yes) (on_board yes)
     (property "Reference" "#PWR0717" (id 0) (at 101.6 134.62 0)
@@
     (pin "4")
   )
-  (symbol (lib_id "power:GND") (at 184.15 143.51 0) (mirror y)
+  (symbol (lib_id "power:GND") (at 184.15 143.51 0) (mirror y) (unit 1)
     (in_bom yes) (on_board yes)
     (property "Reference" "#PWR0722" (id 0) (at 184.15 149.86 0)
@@
     (pin "1")
   )
-  (symbol (lib_id "power:+3.3V") (at 184.15 133.35 0)
+  (symbol (lib_id "power:+3.3V") (at 184.15 133.35 0) (unit 1)
     (in_bom yes) (on_board yes)
     (property "Reference" "#PWR0718" (id 0) (at 184.15 137.16 0)
@@
     (pin "1")
   )
-  (symbol (lib_id "Device:R") (at 237.49 54.61 0) (mirror x)
+  (symbol (lib_id "Device:R") (at 237.49 54.61 0) (mirror x) (unit 1)
     (in_bom yes) (on_board yes)
     (property "Reference" "R702" (id 0) (at 231.775 52.705 0)
@@
     (pin "2")
   )
-  (symbol (lib_id "Device:R") (at 245.11 54.61 0) (mirror x)
+  (symbol (lib_id "Device:R") (at 245.11 54.61 0) (mirror x) (unit 1)
     (in_bom yes) (on_board yes)
     (property "Reference" "R703" (id 0) (at 239.395 52.705 0)
@@
     (pin "2")
   )
-  (symbol (lib_id "power:+3.3V") (at 237.49 49.53 0)
+  (symbol (lib_id "power:+3.3V") (at 237.49 49.53 0) (unit 1)
     (in_bom yes) (on_board yes)
     (property "Reference" "#PWR0706" (id 0) (at 237.49 53.34 0)
@@
     (pin "4")
   )
-  (symbol (lib_id "power:GND") (at 222.25 143.51 0) (mirror y)
+  (symbol (lib_id "power:GND") (at 222.25 143.51 0) (mirror y) (unit 1)
     (in_bom yes) (on_board yes)
     (property "Reference" "#PWR0723" (id 0) (at 222.25 149.86 0)
@@
     (pin "1")
   )
-  (symbol (lib_id "power:+3.3V") (at 222.25 133.35 0)
+  (symbol (lib_id "power:+3.3V") (at 222.25 133.35 0) (unit 1)
     (in_bom yes) (on_board yes)
     (property "Reference" "#PWR0719" (id 0) (at 222.25 137.16 0)
@@
     (pin "1")
   )
-  (symbol (lib_id "power:GND") (at 254 143.51 0)
+  (symbol (lib_id "power:GND") (at 254 143.51 0) (unit 1)
     (in_bom yes) (on_board yes)
     (property "Reference" "#PWR0724" (id 0) (at 254 149.86 0)
@@
     (pin "1")
   )
-  (symbol (lib_id "power:GND") (at 123.825 187.96 0) (mirror y)
+  (symbol (lib_id "power:GND") (at 123.825 187.96 0) (mirror y) (unit 1)
     (in_bom yes) (on_board yes)
     (property "Reference" "#PWR?" (id 0) (at 123.825 194.31 0)
