File: Project/eval_board_tmc6200-ta.kicad_pcb (KiCad board)
At the start: 4 copper layers, 75 x 75 mm, 146 parts, among them J601 Screw_Terminal_01x04, J701 Conn_01x05_Female, J702 Conn_01x04_Female, J703 Conn_01x04_Female, J801 Conn_02x08_Odd_Even, Q201 2N7002, Q301 DMT68M8LFV-7, Q302 DMT68M8LFV-7, Q401 DMT68M8LFV-7, Q402 DMT68M8LFV-7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

Commit message: Cleanup ED A1 version
Parts:
- removed REF**: WEEE-Logo_4.2x6mm_SilkScreen, Symbol:WEEE-Logo_4.2x6mm_SilkScreen
- removed REF**: ESD-Logo_6.6x6mm_SilkScreen, Symbol:ESD-Logo_6.6x6mm_SilkScreen
- removed REF**: OSHW-Logo2_7.3x6mm_SilkScreen, Symbol:OSHW-Logo2_7.3x6mm_SilkScreen
Connections:
- net /BLDC_MOTOR.sch/+12V_INTERNAL renamed /BLDC_MOTOR/+12V_INTERNAL
- net /BLDC_MOTOR.sch/+5V_INTERNAL renamed /BLDC_MOTOR/+5V_INTERNAL
- net /BLDC_MOTOR.sch/CONN_U renamed /BLDC_MOTOR/CONN_U
- net /BLDC_MOTOR.sch/CONN_V renamed /BLDC_MOTOR/CONN_V
- net /BLDC_MOTOR.sch/CONN_W renamed /BLDC_MOTOR/CONN_W
- net /BLDC_MOTOR.sch/HSU renamed /BLDC_MOTOR/HSU
- net /BLDC_MOTOR.sch/HSV renamed /BLDC_MOTOR/HSV
- net /BLDC_MOTOR.sch/HSW renamed /BLDC_MOTOR/HSW
- net /BLDC_MOTOR.sch/IC_CLK renamed /BLDC_MOTOR/IC_CLK
- net /BLDC_MOTOR.sch/IC_CSN renamed /BLDC_MOTOR/IC_CSN
- net /BLDC_MOTOR.sch/IC_CURU renamed /BLDC_MOTOR/IC_CURU
- net /BLDC_MOTOR.sch/IC_CURV renamed /BLDC_MOTOR/IC_CURV
- net /BLDC_MOTOR.sch/IC_CURW renamed /BLDC_MOTOR/IC_CURW
- net /BLDC_MOTOR.sch/IC_DRV_EN renamed /BLDC_MOTOR/IC_DRV_EN
- net /BLDC_MOTOR.sch/IC_FAULT renamed /BLDC_MOTOR/IC_FAULT
- net /BLDC_MOTOR.sch/IC_SCK renamed /BLDC_MOTOR/IC_SCK
- net /BLDC_MOTOR.sch/IC_SDI renamed /BLDC_MOTOR/IC_SDI
- net /BLDC_MOTOR.sch/IC_SDO renamed /BLDC_MOTOR/IC_SDO
- net /BLDC_MOTOR.sch/IC_SPE_CTRL renamed /BLDC_MOTOR/IC_SPE_CTRL
- net /BLDC_MOTOR.sch/IC_STD_ALONE renamed /BLDC_MOTOR/IC_STD_ALONE
- net /BLDC_MOTOR.sch/IC_VOFS_TEST renamed /BLDC_MOTOR/IC_VOFS_TEST
- net /BLDC_MOTOR.sch/LSU renamed /BLDC_MOTOR/LSU
- net /BLDC_MOTOR.sch/LSV renamed /BLDC_MOTOR/LSV
- net /BLDC_MOTOR.sch/LSW renamed /BLDC_MOTOR/LSW
- net /BLDC_MOTOR.sch/STAND1 renamed /BLDC_MOTOR/STAND1
- net /BLDC_MOTOR.sch/STAND2 renamed /BLDC_MOTOR/STAND2
- net /BLDC_MOTOR.sch/STAND3 renamed /BLDC_MOTOR/STAND3
- net /BLDC_MOTOR.sch/STAND4 renamed /BLDC_MOTOR/STAND4
- net /BLDC_MOTOR.sch/STAND5 renamed /BLDC_MOTOR/STAND5
- net /BLDC_MOTOR.sch/STAND6 renamed /BLDC_MOTOR/STAND6
- net /BLDC_MOTOR.sch/U renamed /BLDC_MOTOR/U
- net /BLDC_MOTOR.sch/USENSE renamed /BLDC_MOTOR/USENSE
- net /BLDC_MOTOR.sch/V renamed /BLDC_MOTOR/V
- net /BLDC_MOTOR.sch/VCC_IO renamed /BLDC_MOTOR/VCC_IO
- net /BLDC_MOTOR.sch/VSENSE renamed /BLDC_MOTOR/VSENSE
- net /BLDC_MOTOR.sch/W renamed /BLDC_MOTOR/W
- net /BLDC_MOTOR.sch/WSENSE renamed /BLDC_MOTOR/WSENSE
- net /BUCK_Converter.sch/RESET_3V3 renamed /Microcontroller/RESET_3V3
- net /IO Expander.sch/EXP_INT_A renamed /IO Expander/EXP_INT_1
- net /IO Expander.sch/EXP_INT_B renamed /IO Expander/EXP_INT_2
- net /IO Expander.sch/GPA0 renamed /IO Expander/GPA0
- net /IO Expander.sch/GPA1 renamed /IO Expander/GPA1
- net /IO Expander.sch/GPA2 renamed /IO Expander/GPA2
- net /IO Expander.sch/GPA3 renamed /IO Expander/GPA3
- net /IO Expander.sch/GPA4 renamed /IO Expander/GPA4
- net /IO Expander.sch/GPA5 renamed /IO Expander/GPA5
- net /IO Expander.sch/GPA6 renamed /IO Expander/GPA6
- net /IO Expander.sch/GPA7 renamed /IO Expander/GPA7
- net /IO Expander.sch/IN_A0 renamed /IO Expander/IN_A0
- net /IO Expander.sch/IN_A1 renamed /IO Expander/IN_A1
- net /IO Expander.sch/IN_A2 renamed /IO Expander/IN_A2
- net /IO Expander.sch/IN_A3 renamed /IO Expander/IN_A3
- net /IO Expander.sch/IN_A4 renamed /IO Expander/IN_A4
- net /IO Expander.sch/IN_A5 renamed /IO Expander/IN_A5
- net /IO Expander.sch/IN_A6 renamed /IO Expander/IN_A6
- net /IO Expander.sch/IN_A7 renamed /IO Expander/IN_A7
- net /Microcontroller.sch/HEART_BIT_LED renamed /Microcontroller/HEART_BIT_LED
- net /Microcontroller.sch/SWCLK renamed /Microcontroller/SWCLK
- net /Microcontroller.sch/SWDIO renamed /Microcontroller/SWDIO
- net /Microcontroller.sch/USART2_RX renamed /Microcontroller/USART2_RX
- net /Microcontroller.sch/USART2_TX renamed /Microcontroller/USART2_TX
- C706 pad 1: RESET -> /Microcontroller/RESET
- H701 pad 1: Net-(H701-Pad1) -> unconnected-(H701-Pad1)
- H703 pad 1: Net-(H703-Pad1) -> unconnected-(H703-Pad1)
- H704 pad 1: Net-(H704-Pad1) -> unconnected-(H704-Pad1)
- J701 pad 4: RESET -> /Microcontroller/RESET
- J702 pad 3: /IO Expander.sch/I2C1_SDA -> /Microcontroller/I2C1_SDA
- J702 pad 4: /IO Expander.sch/I2C1_SCL -> /Microcontroller/I2C1_SCL
- R702 pad 1: /IO Expander.sch/I2C1_SDA -> /Microcontroller/I2C2
- R703 pad 1: /IO Expander.sch/I2C1_SCL -> /Microcontroller/I2C1
- R704 pad 1: RESET -> /Microcontroller/RESET
- U201 pad 2: Net-(U201-Pad2) -> unconnected-(U201-Pad2)
- U201 pad 28: Net-(U201-Pad28) -> unconnected-(U201-Pad28)
- U201 pad 31: Net-(U201-Pad31) -> unconnected-(U201-Pad31)
- U201 pad 35: Net-(U201-Pad35) -> unconnected-(U201-Pad35)
- U201 pad 40: Net-(U201-Pad40) -> unconnected-(U201-Pad40)
- U201 pad 45: Net-(U201-Pad45) -> unconnected-(U201-Pad45)
- U701 pad 14: Net-(U701-Pad14) -> unconnected-(U701-Pad14)
- U701 pad 16: Net-(U701-Pad16) -> unconnected-(U701-Pad16)
- U701 pad 18: Net-(U701-Pad18) -> unconnected-(U701-Pad18)
- U701 pad 19: /IO Expander.sch/I2C1_SDA -> /Microcontroller/I2C2
- U701 pad 2: Net-(U701-Pad2) -> unconnected-(U701-Pad2)
- U701 pad 20: /IO Expander.sch/I2C1_SCL -> /Microcontroller/I2C1
- U701 pad 3: Net-(U701-Pad3) -> unconnected-(U701-Pad3)
- U701 pad 4: RESET -> /Microcontroller/RESET
- U701 pad 9: Net-(U701-Pad9) -> unconnected-(U701-Pad9)
- U801 pad 10: Net-(U801-Pad10) -> unconnected-(U801-Pad10)
- U801 pad 3: Net-(U801-Pad3) -> unconnected-(U801-Pad3)
- U801 pad 4: Net-(U801-Pad4) -> unconnected-(U801-Pad4)
- U801 pad 7: Net-(U801-Pad7) -> unconnected-(U801-Pad7)
- U801 pad 8: /IO Expander.sch/I2C1_SCL -> /IO Expander/I2C1
- U801 pad 9: /IO Expander.sch/I2C1_SDA -> /IO Expander/I2C2
Routing:
- net RESET: track 74.0 -> 0.00 mm, vias 3 -> 0
- net /Microcontroller/RESET: track 0.00 -> 74.0 mm, vias 0 -> 3
- net /IO Expander.sch/I2C1_SCL: track 59.0 -> 0.00 mm, vias 2 -> 0
- net /IO Expander.sch/I2C1_SDA: track 58.9 -> 0.00 mm, vias 2 -> 0
- net /Microcontroller/I2C1_SCL: track 0.00 -> 30.7 mm, vias 0 -> 1
- net /Microcontroller/I2C1_SDA: track 0.00 -> 30.5 mm, vias 0 -> 1
